Commit message: Added camera, microphone and rest of ultrasonic sensors to urdf

File: description/robot.urdf.xacro (robot description, xacro)
@@ -2,4 +2,9 @@
 <robot xmlns:xacro="http://www.ros.org/wiki/xacro" name="robot">
     <xacro:include filename="robot_core.xacro" />
-    <xacro:include filename="ultrasonic.xacro" />
+    <xacro:include filename="ultrasonic_front.xacro" />
+    <xacro:include filename="ultrasonic_bottom_front.xacro" />
+    <xacro:include filename="ultrasonic_back.xacro" />
+    <xacro:include filename="ultrasonic_bottom_back.xacro" />
+    <xacro:include filename="camera.xacro" />
+    <xacro:include filename="microphone.xacro" />
 </robot>

File: description/ultrasonic_bottom_back.xacro (robot description, xacro)
@@ -2,25 +2,25 @@
 <robot xmlns:xacro="http://www.ros.org/wiki/xacro">
     <xacro:include filename="inertia_macros.xacro" />
-    <joint name="ultrasonic_front_joint" type="fixed">
+    <joint name="ultrasonic_bottom_back_joint" type="fixed">
         <parent link="chassis" />
-        <child link="ultrasonic_front" />
+        <child link="ultrasonic_bottom_back" />
         <origin xyz="0 0.205 0.125" />
     </joint>
-    <link name="ultrasonic_front">
+    <link name="ultrasonic_bottom_back">
         <visual>
-            <origin xyz="-0.01 -0.01 -0.07" rpy="${-pi/2} 0 ${pi/2}" />
+            <origin xyz="-0.01 -0.29 -0.1" rpy="${pi/2} ${pi/11} ${pi/2}" />
             <geometry>
                 <mesh filename="package://fonbot_package/models/ultrasonic.dae" scale="0.3 0.3 0.3" />
             </geometry>
-            <material name="black" />
         </visual>
         <collision>
+            <origin xyz="-0.01 -0.4 -0.077" rpy="${pi/2} ${7*pi/12} ${pi/2}" />
             <geometry>
-                <box size="0.2 0.2 0.2" />
+                <mesh filename="package://fonbot_package/models/ultrasonic.dae" scale="0.3 0.3 0.3" />
             </geometry>
         </collision>
-        <xacro:inertial_box mass="0.05" x="0.2" y="0.2" z="0.2">
+        <!-- <xacro:inertial_box mass="0.05" x="0.2" y="0.2" z="0.2">
             <origin xyz="0 0 0" rpy="0 0 0" />
-        </xacro:inertial_box>
+        </xacro:inertial_box> -->
     </link>
 </robot>
